Commit message: Modified package name
Signed-off-by: daveohs <wellclosedoor@gmail.com>

File: urdf/manipulator.urdf (robot description, URDF)
Before this commit: robot my_manipulator, 8 links, 7 joints
Links:
- link link_1: geometry collision mesh filename=package://manipulator/meshes/link_1.stl scale=0.001 0.001 0.001; visual mesh filename=package://manipulator/meshes/link_1.stl scale=0.001 0.001 0.001
- link link_2: geometry collision mesh filename=package://manipulator/meshes/link_2.stl scale=0.001 0.001 0.001; visual mesh filename=package://manipulator/meshes/link_2.stl scale=0.001 0.001 0.001
- link link_3: geometry collision mesh filename=package://manipulator/meshes/link_3.stl scale=0.001 0.001 0.001; visual mesh filename=package://manipulator/meshes/link_3.stl scale=0.001 0.001 0.001
- link link_4: geometry collision mesh filename=package://manipulator/meshes/link_4.stl scale=0.001 0.001 0.001; visual mesh filename=package://manipulator/meshes/link_4.stl scale=0.001 0.001 0.001
- link link_5: geometry collision mesh filename=package://manipulator/meshes/link_5.stl scale=0.001 0.001 0.001; visual mesh filename=package://manipulator/meshes/link_5.stl scale=0.001 0.001 0.001
- link link_6: geometry collision mesh filename=package://manipulator/meshes/link_6.stl scale=0.001 0.001 0.001; visual mesh filename=package://manipulator/meshes/link_6.stl scale=0.001 0.001 0.001
- link link_7: geometry collision mesh filename=package://manipulator/meshes/link_7.stl scale=0.001 0.001 0.001; visual mesh filename=package://manipulator/meshes/link_7.stl scale=0.001 0.001 0.001
